File: elec/layout/default/swoop.kicad_pcb (KiCad board)
At the start: 2 copper layers, 225.7 x 100.8 mm, 0 parts

Commit message: checkin
Parts:
- added C1: 50V 20pF C0G ±5% 0402 Multilayer Ceramic Capacitors MLCC - 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, lib:C0402, F.Cu at (160.7, 99.5)
- added C10: 16V 100nF X7R ±10% 0402 Multilayer Ceramic Capacitors MLCC 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, lib:C0402, F.Cu at (170.1, 87.4)
- added C11: 16V 100nF X7R ±10% 0402 Multilayer Ceramic Capacitors MLCC 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, lib:C0402, F.Cu at (167.1, 98.3)
- added C12: 25V 1uF X5R ±10% 0402 Multilayer Ceramic Capacitors MLCC - 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, lib:C0402, F.Cu at (168.1, 98.3)
- added C13: Multilayer Ceramic Capacitors MLCC - SMD/SMT 1uF 6.3V 0402 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, lib:C0402, F.Cu at (165.7, 116.4)
- added C14: Multilayer Ceramic Capacitors MLCC - SMD/SMT 1uF 6.3V 0402 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, lib:C0402, F.Cu at (162.3, 116.4)
- added C15: Multilayer Ceramic Capacitors MLCC - SMD/SMT 10uF 10V 0805 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, lib:C0805, F.Cu at (135.7, 61.5)
- added C16: Multilayer Ceramic Capacitors MLCC - SMD/SMT 10uF 10V 0805 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, lib:C0805, F.Cu at (135.7, 59.5)
- added C17: Multilayer Ceramic Capacitors MLCC - SMD/SMT 10uF 10V 0805 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, lib:C0805, F.Cu at (135.6, 68.7)
- added C18: Multilayer Ceramic Capacitors MLCC - SMD/SMT 10uF 10V 0805 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, lib:C0805, F.Cu at (135.6, 70.7)
- added C19: Multilayer Ceramic Capacitors MLCC - SMD/SMT 100nF 10V 0402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, lib:C0402, F.Cu at (132.8, 66.2)
- added C2: 50V 20pF C0G ±5% 0402 Multilayer Ceramic Capacitors MLCC - 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, lib:C0402, F.Cu at (166.0, 100.2)
- added C20: Multilayer Ceramic Capacitors MLCC - SMD/SMT 10uF 10V 0805 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, lib:C0805, F.Cu at (133.4, 111.4)
- added C21: Multilayer Ceramic Capacitors MLCC - SMD/SMT 10uF 10V 0805 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, lib:C0805, F.Cu at (133.2, 120.4)
- added C22: 16V 100nF X7R ±10% 0402 Multilayer Ceramic Capacitors MLCC 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, lib:C0402, F.Cu at (136.2, 96.5)
- added C23: 25V 1uF X5R ±10% 0402 Multilayer Ceramic Capacitors MLCC - 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, lib:C0402, F.Cu at (134.2, 96.5)
- added C24: 16V 100nF X7R ±10% 0402 Multilayer Ceramic Capacitors MLCC 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, lib:C0402, F.Cu at (138.9, 93.6)
- added C25: 50V 22pF C0G ±5% 0402 Multilayer Ceramic Capacitors MLCC - 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, lib:C0402, F.Cu at (130.4, 97.1)
- added C26: 50V 22pF C0G ±5% 0402 Multilayer Ceramic Capacitors MLCC - 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, lib:C0402, F.Cu at (130.4, 92.0)
- added C27: 16V 100nF X7R ±10% 0402 Multilayer Ceramic Capacitors MLCC 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, lib:C0402, F.Cu at (162.8, 64.8)
- added C28: 16V 100nF X7R ±10% 0402 Multilayer Ceramic Capacitors MLCC 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, lib:C0402, F.Cu at (167.9, 66.3)
- added C29: 16V 100nF X7R ±10% 0402 Multilayer Ceramic Capacitors MLCC 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, lib:C0402, F.Cu at (183.5, 63.2)
- added C3: 16V 100nF X7R ±10% 0402 Multilayer Ceramic Capacitors MLCC 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, lib:C0402, F.Cu at (166.0, 98.3)
- added C30: 25V 1uF X5R ±10% 0402 Multilayer Ceramic Capacitors MLCC - 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, lib:C0402, F.Cu at (183.5, 62.2)
- added C31: 16V 100nF X7R ±10% 0402 Multilayer Ceramic Capacitors MLCC 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, lib:C0402, F.Cu at (179.8, 60.1)
- added C4: 16V 100nF X7R ±10% 0402 Multilayer Ceramic Capacitors MLCC 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, lib:C0402, F.Cu at (170.1, 88.5)
- added C5: 16V 100nF X7R ±10% 0402 Multilayer Ceramic Capacitors MLCC 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, lib:C0402, F.Cu at (159.4, 87.4)
- added C6: 16V 100nF X7R ±10% 0402 Multilayer Ceramic Capacitors MLCC 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, lib:C0402, F.Cu at (159.4, 88.5)
- added C7: 16V 100nF X7R ±10% 0402 Multilayer Ceramic Capacitors MLCC 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, lib:C0402, F.Cu at (170.2, 92.3)
- added C8: 25V 1uF X5R ±10% 0402 Multilayer Ceramic Capacitors MLCC - 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, lib:C0402, F.Cu at (168.4, 79.2)
- added C9: 16V 100nF X7R ±10% 0402 Multilayer Ceramic Capacitors MLCC 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, lib:C0402, F.Cu at (164.7, 86.0)
- added L1: , lib:IND-SMD_L2.5-W2.0_WPN252012H, F.Cu at (139.9, 64.8)
- added LED1: , lib:LED0603-RD, F.Cu at (161.0, 118.8)
- added LED2: , lib:LED0603-RD, F.Cu at (161.0, 115.8)
- added R1: 62.5mW Thick Film Resistors ±100ppm/℃ ±1% 1kΩ 0402 Chip Res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, lib:R0402, F.Cu at (164.5, 97.2)
- added R10: Chip Resistor - Surface Mount 180KOhms ±5% 1/16W 0402 RoHS, lib:R0402, F.Cu at (134.4, 67.2)
- added R11: Chip Resistor - Surface Mount 1MOhms ±5% 1/16W 0402 RoHS, lib:R0402, F.Cu at (132.9, 63.2)
- added R12: 62.5mW Thick Film Resistors ±100ppm/℃ ±1% 10kΩ 0402 Chip Re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, lib:R0402, F.Cu at (136.2, 89.4)
- added R13: 62.5mW Thick Film Resistors ±100ppm/℃ ±1% 10kΩ 0402 Chip Re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, lib:R0402, F.Cu at (138.9, 94.7)
- added R14: 62.5mW Thick Film Resistors ±100ppm/℃ ±1% 10kΩ 0402 Chip Re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, lib:R0402, F.Cu at (138.9, 95.8)
- added R15: 62.5mW Thick Film Resistors ±100ppm/℃ ±1% 1kΩ 0402 Chip Res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, lib:R0402, F.Cu at (180.8, 60.1)
- added R16: 62.5mW Thick Film Resistors ±100ppm/℃ ±1% 5.1kΩ 0402 Chip R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, lib:R0402, F.Cu at (104.0, 92.6)
- added R17: 62.5mW Thick Film Resistors ±100ppm/℃ ±1% 5.1kΩ 0402 Chip R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, lib:R0402, F.Cu at (98.4, 94.4)
- added R18: 62.5mW Thick Film Resistors ±100ppm/℃ ±1% 10kΩ 0402 Chip Re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, lib:R0402, F.Cu at (108.9, 92.6)
- added R19: 62.5mW Thick Film Resistors ±100ppm/℃ ±1% 10kΩ 0402 Chip Re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, lib:R0402, F.Cu at (104.0, 88.6)
- added R2: 62.5mW Thick Film Resistors ±100ppm/℃ ±1% 27kΩ 0402 Chip Re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, lib:R0402, F.Cu at (168.4, 85.3)
- added R20: 62.5mW Thick Film Resistors ±100ppm/℃ ±1% 10kΩ 0402 Chip Re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, lib:R0402, F.Cu at (104.0, 96.6)
- added R21: 62.5mW Thick Film Resistors ±100ppm/℃ ±1% 10kΩ 0402 Chip Re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, lib:R0402, F.Cu at (108.9, 88.6)
- added R3: 62.5mW Thick Film Resistors ±100ppm/℃ ±1% 27kΩ 0402 Chip Re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, lib:R0402, F.Cu at (168.4, 86.4)
- added R4: 62.5mW Thick Film Resistors ±100ppm/℃ ±1% 10kΩ 0402 Chip Re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, lib:R0402, F.Cu at (159.4, 92.3)
- added R5: 62.5mW Thick Film Resistors ±100ppm/℃ ±1% 10kΩ 0402 Chip Re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, lib:R0402, F.Cu at (161.4, 86.4)
- added R6: 62.5mW Thick Film Resistors ±100ppm/℃ ±1% 510Ω 0402 Chip Re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, lib:R0402, F.Cu at (162.3, 118.3)
- added R7: Chip Resistor - Surface Mount 120Ohms ±5% 1/16W 0402 RoHS, lib:R0402, F.Cu at (162.8, 119.8)
- added R8: Chip Resistor - Surface Mount 82Ohms ±5% 1/16W 0402 RoHS, lib:R0402, F.Cu at (162.8, 115.0)
- added R9: Chip Resistor - Surface Mount 1MOhms ±5% 1/16W 0402 RoHS, lib:R0402, F.Cu at (136.3, 67.2)
- added U1: , lib:LQFN-56_L7.0-W7.0-P0.4-EP, F.Cu at (164.7, 91.3)
- added U10: , lib:LGA-16_L4.5-W3.0-P0.50-BL, F.Cu at (165.3, 66.3)
- added U11: , lib:LGA-12_L2.0-W2.0-P0.50-BL, F.Cu at (181.0, 62.5)
- added U12: , lib:USB-C-SMD_KH-TYPE-C-16P, F.Cu at (90.7, 83.9)
- added U2: , lib:OSC-SMD_4P-L3.2-W2.5-BL, F.Cu at (163.3, 99.5)
- added U3: , lib:SOIC-8_L5.3-W5.3-P1.27-LS8.0-BL, F.Cu at (164.7, 82.3)
- added U4: , lib:CONN-SMD_P2.00_S2B-PH-SM4-TB-LF-SN, F.Cu at (179.5, 116.5)
- added U5: , lib:WSON-10_L2.0-W2.0-P0.40-BL-EP, F.Cu at (164.0, 117.2)
- added U6: , lib:VSON-14_L4.0-W3.0-P0.50-BL-EP_TI_DSJ, F.Cu at (136.2, 64.7)
- added U7: , lib:SOT-223-3_L6.5-W3.4-P2.30-LS7.0-BR, F.Cu at (133.4, 115.9)
- added U8: , lib:LGA-28_L5.2-W3.8-P0.50-BL, F.Cu at (135.3, 93.0)
- added U9: , lib:FC-135R_L3.2-W1.5, F.Cu at (130.4, 94.5)
Routing:
- net vcc: track 0.00 -> 71.7 mm, vias 0 -> 3
- net gnd: track 0.00 -> 45.2 mm, vias 0 -> 2
- net vcc-1: track 0.00 -> 23.4 mm, vias 0 -> 2
- net sck: track 0.00 -> 14.4 mm
- net io0: track 0.00 -> 12.8 mm, vias 0 -> 2
- net vcc-4: track 0.00 -> 10.1 mm
- net vcc-3: track 0.00 -> 9.80 mm
- net io3: track 0.00 -> 9.73 mm
- net io1: track 0.00 -> 9.57 mm
- net cs: track 0.00 -> 9.55 mm
- net xin: track 0.00 -> 8.08 mm
- net io2: track 0.00 -> 6.20 mm
- net vcc-2: track 0.00 -> 6.03 mm, vias 0 -> 2
- net xin32: track 0.00 -> 5.61 mm
- net xout32: track 0.00 -> 5.04 mm
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Other:
- board size 225.7 x 100.8 mm -> 100 x 100 mm
