File: elec/layout/default/swoop.kicad_pcb (KiCad board)
At the start: 2 copper layers, 100 x 100 mm, 80 parts

Commit message: merging in layouts
Parts:
- removed LED1, LED2: , lib:LED0603-RD
- added C36: 25V 10uF X5R ±10% 0805 Multilayer Ceramic Capacitors MLCC -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, lib:C0805, F.Cu at (164.9, 120.8)
- added C37: 25V 10uF X5R ±10% 0805 Multilayer Ceramic Capacitors MLCC -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, lib:C0805, F.Cu at (165.0, 122.8)
- added C38: 50V 11pF C0G ±5% 0402 Multilayer Ceramic Capacitors MLCC - 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, lib:C0402, F.Cu at (172.9, 133.2)
- added C39: 50V 11pF C0G ±5% 0402 Multilayer Ceramic Capacitors MLCC - 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, lib:C0402, F.Cu at (177.6, 132.7)
- added C40: 10V 470nF X5R ±10% 0402 Multilayer Ceramic Capacitors MLCC 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, lib:C0402, F.Cu at (170.3, 132.8)
- added C41: 16V 100nF X7R ±10% 0402 Multilayer Ceramic Capacitors MLCC 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, lib:C0402, F.Cu at (174.0, 124.4)
- added C42: 16V 100nF X7R ±10% 0402 Multilayer Ceramic Capacitors MLCC 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, lib:C0402, F.Cu at (177.1, 127.0)
- added C43: 50V 10nF X7R ±10% 0402 Multilayer Ceramic Capacitors MLCC -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, lib:C0402, F.Cu at (177.1, 126.1)
- added C44: 50V 10nF X7R ±10% 0402 Multilayer Ceramic Capacitors MLCC -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, lib:C0402, F.Cu at (170.3, 131.8)
- added C45: 50V 1pF C0G 0402 Multilayer Ceramic Capacitors MLCC - SMD/S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, lib:C0402, F.Cu at (170.2, 126.8)
- added C46: 50V 1pF C0G 0402 Multilayer Ceramic Capacitors MLCC - SMD/S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, lib:C0402, F.Cu at (169.5, 129.6)
- added C47: 50V 1pF C0G 0402 Multilayer Ceramic Capacitors MLCC - SMD/S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, lib:C0402, F.Cu at (166.7, 129.6)
- added C48: 50V 1pF C0G 0402 Multilayer Ceramic Capacitors MLCC - SMD/S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, lib:C0402, F.Cu at (168.1, 129.2)
- added C49: 50V 100pF C0G ±5% 0402 Multilayer Ceramic Capacitors MLCC -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, lib:C0402, F.Cu at (166.3, 128.2)
- added C50: 16V 100nF X7R ±10% 0402 Multilayer Ceramic Capacitors MLCC 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, lib:C0402, F.Cu at (157.2, 49.0)
- added C51: 16V 100nF X7R ±10% 0402 Multilayer Ceramic Capacitors MLCC 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, lib:C0402, F.Cu at (124.8, 34.0)
- added C52: 16V 100nF X7R ±10% 0402 Multilayer Ceramic Capacitors MLCC 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, lib:C0402, F.Cu at (118.5, 31.0)
- added C53: 16V 100nF X7R ±10% 0402 Multilayer Ceramic Capacitors MLCC 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, lib:C0402, F.Cu at (112.6, 28.4)
- added C54: 16V 100nF X7R ±10% 0402 Multilayer Ceramic Capacitors MLCC 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, lib:C0402, F.Cu at (135.7, 46.0)
- added C55: 16V 100nF X7R ±10% 0402 Multilayer Ceramic Capacitors MLCC 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, lib:C0402, F.Cu at (132.6, 45.0)
- added C56: 25V 1uF X5R ±10% 0402 Multilayer Ceramic Capacitors MLCC - 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, lib:C0402, F.Cu at (174.9, 92.8)
- added C57: 25V 1uF X5R ±10% 0402 Multilayer Ceramic Capacitors MLCC - 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, lib:C0402, F.Cu at (176.9, 92.8)
- added J1: , lib:CONN-SMD_4P-P1.00_SM04B-SRSS-TB-LF-SN, F.Cu at (159.8, 151.7)
- added J2: , lib:CONN-SMD_4P-P1.00_SM04B-SRSS-TB-LF-SN, F.Cu at (165.1, 64.8)
- added L2: , lib:L0402, F.Cu at (170.0, 128.2)
- added L3: , lib:L0402, F.Cu at (168.1, 128.2)
- added R23: 62.5mW Thick Film Resistors ±100ppm/℃ ±1% 5.1kΩ 0402 Chip R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, lib:R0402, F.Cu at (175.9, 84.1)
- added R24: 62.5mW Thick Film Resistors ±100ppm/℃ ±1% 10kΩ 0402 Chip Re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, lib:R0402, F.Cu at (162.4, 70.5)
- added R25: 62.5mW Thick Film Resistors ±100ppm/℃ ±1% 10kΩ 0402 Chip Re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, lib:R0402, F.Cu at (161.3, 70.5)
- added R26: 62.5mW Thick Film Resistors ±100ppm/℃ ±1% 10kΩ 0402 Chip Re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, lib:R0402, F.Cu at (184.2, 102.4)
- added R27: 62.5mW Thick Film Resistors ±100ppm/℃ ±1% 5.1kΩ 0402 Chip R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, lib:R0402, F.Cu at (168.5, 146.7)
- added R28: 62.5mW Thick Film Resistors ±100ppm/℃ ±1% 5.1kΩ 0402 Chip R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, lib:R0402, F.Cu at (171.5, 146.6)
- added R29: 62.5mW Thick Film Resistors ±100ppm/℃ ±1% 10kΩ 0402 Chip Re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, lib:R0402, F.Cu at (152.0, 46.7)
- added R30: 62.5mW Thick Film Resistors ±100ppm/℃ ±1% 10kΩ 0402 Chip Re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, lib:R0402, F.Cu at (171.8, 54.6)
- added R31: 62.5mW Thick Film Resistors ±100ppm/℃ ±1% 3.24kΩ 0402 Chip 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, lib:R0402, F.Cu at (132.6, 43.2)
- added U21: , lib:LGA-16_L4.5-W3.0-P0.50-BL, F.Cu at (179.1, 76.2)
- added U22: , lib:QFN-24_L4.0-W4.0-P0.50-BL-EP2.7, F.Cu at (169.9, 84.9)
- added U23: , lib:LGA-12_L2.0-W2.0-P0.50-BL, F.Cu at (138.6, 151.6)
- added U24: , lib:WIRELM-SMD_ESP32-S3-WROOM-1, F.Cu at (172.6, 108.4)
- added U25: , lib:KEY-SMD_4P-L4.2-W3.2-P2.20-LS4.6, F.Cu at (169.8, 121.8)
- added U26: , lib:QFN-24_L4.0-W4.0-P0.50-BL-EP2.6, F.Cu at (173.6, 127.9)
- added U27: , lib:OSC-SMD_4P-L2.0-W1.6-BL, F.Cu at (175.3, 132.6)
- added U28: , lib:IPEX-SMD_BWIPX-1-001E, F.Cu at (163.8, 128.3)
- added U29: , lib:USB-C-SMD_KH-TYPE-C-16P, F.Cu at (180.7, 85.4)
- added U30: , lib:KEY-SMD_4P-L4.2-W3.2-P2.20-LS4.6, F.Cu at (184.9, 106.1)
- added U31: , lib:HDR-SMD_10P-P1.27-V-M-R2-C5-LS5.3, F.Cu at (168.8, 94.3)
- added U32: , lib:USB-C-SMD_KH-TYPE-C-16P, F.Cu at (169.7, 151.2)
- added U33: , lib:LED-SMD_4P-L2.0-W2.0-BR, F.Cu at (157.9, 47.1)
- added U34: , lib:LED-SMD_4P-L2.0-W2.0-BR, F.Cu at (125.6, 32.0)
- added U35: , lib:LED-SMD_4P-L2.0-W2.0-BR, F.Cu at (119.3, 29.0)
- added U36: , lib:LED-SMD_4P-L2.0-W2.0-BR, F.Cu at (113.4, 26.4)
- added U37: , lib:SW-TH_TS-1093C-A7B3-D1, F.Cu at (146.9, 45.4)
- added U38: , lib:SW-TH_TS-1093C-A7B3-D1, F.Cu at (166.2, 53.7)
- added U39: , lib:SOT-23-3_L2.9-W1.3-P0.95-LS2.4-BR, F.Cu at (134.6, 44.1)
- added U40: , lib:VSSOP-10_L3.0-W3.0-P0.50-LS4.9-BL, F.Cu at (176.0, 95.1)
- added U41: , lib:CONN-TH_DB125-2.54-2P-GN, F.Cu at (182.9, 94.8)
- C23, C30: value 25V 1uF X5R ±10% 0402 Multilayer Ceramic Capacitors MLCC - SMD/SMT ROHS -> 16V 100nF X7R ±10% 0402 Multilayer Ceramic Capacitors MLCC - SMD/SMT ROHS
- C24, C33: value 16V 100nF X7R ±10% 0402 Multilayer Ceramic Capacitors MLCC - SMD/SMT ROHS -> 25V 1uF X5R ±10% 0402 Multilayer Ceramic Capacitors MLCC - SMD/SMT ROHS
- C25: value 50V 22pF C0G ±5% 0402 Multilayer Ceramic Capacitors MLCC - SMD/SMT ROHS -> 16V 100nF X7R ±10% 0402 Multilayer Ceramic Capacitors MLCC - SMD/SMT ROHS
- C27: value 16V 100nF X7R ±10% 0402 Multilayer Ceramic Capacitors MLCC - SMD/SMT ROHS -> 50V 22pF C0G ±5% 0402 Multilayer Ceramic Capacitors MLCC - SMD/SMT ROHS
- C31: value 16V 100nF X7R ±10% 0402 Multilayer Ceramic Capacitors MLCC - SMD/SMT ROHS -> 50V 2.2nF X7R ±10% 0603 Multilayer Ceramic Capacitors MLCC - SMD/SMT ROHS; footprint lib:C0402 -> lib:C0603
- R1: value 62.5mW Thick Film Resistors ±100ppm/℃ ±1% 1kΩ 0402 Chip Resistor - Surface Mount ROHS -> 62.5mW Thick Film Resistors ±100ppm/℃ ±1% 10kΩ 0402 Chip Resistor - Surface Mount ROHS
- R10: value 62.5mW Thick Film Resistors ±100ppm/℃ ±1% 180kΩ 0402 Chip Resistor - Surface Mount ROHS -> 62.5mW Thick Film Resistors ±100ppm/℃ ±1% 105kΩ 0402 Chip Resistor - Surface Mount ROHS
- R12: value 62.5mW Thick Film Resistors ±100ppm/℃ ±1% 10kΩ 0402 Chip Resistor - Surface Mount ROHS -> 62.5mW Thick Film Resistors ±100ppm/℃ ±1% 16.2kΩ 0402 Chip Resistor - Surface Mount ROHS
- R13: value 62.5mW Thick Film Resistors ±100ppm/℃ ±1% 10kΩ 0402 Chip Resistor - Surface Mount ROHS -> 62.5mW Thick Film Resistors ±100ppm/℃ ±1% 17.8kΩ 0402 Chip Resistor - Surface Mount ROHS
- R14: value 62.5mW Thick Film Resistors ±100ppm/℃ ±1% 10kΩ 0402 Chip Resistor - Surface Mount ROHS -> 62.5mW Thick Film Resistors ±1% ±400ppm/℃ 5.1Ω 0402 Chip Resistor - Surface Mount ROHS
- R15: value 62.5mW Thick Film Resistors ±100ppm/℃ ±1% 1kΩ 0402 Chip Resistor - Surface Mount ROHS -> 62.5mW Thick Film Resistors ±1% ±400ppm/℃ 5.1Ω 0402 Chip Resistor - Surface Mount ROHS
- R16: value 62.5mW Thick Film Resistors ±100ppm/℃ ±1% 5.1kΩ 0402 Chip Resistor - Surface Mount ROHS -> 62.5mW Thick Film Resistors ±1% ±400ppm/℃ 5.1Ω 0402 Chip Resistor - Surface Mount ROHS
- R17: value 62.5mW Thick Film Resistors ±100ppm/℃ ±1% 5.1kΩ 0402 Chip Resistor - Surface Mount ROHS -> 62.5mW Thick Film Resistors ±100ppm/℃ ±1% 10kΩ 0402 Chip Resistor - Surface Mount ROHS
- R2: value 62.5mW Thick Film Resistors ±100ppm/℃ ±1% 27kΩ 0402 Chip Resistor - Surface Mount ROHS -> 62.5mW Thick Film Resistors ±100ppm/℃ ±1% 10kΩ 0402 Chip Resistor - Surface Mount ROHS
- R20: value 62.5mW Thick Film Resistors ±100ppm/℃ ±1% 10kΩ 0402 Chip Resistor - Surface Mount ROHS -> 62.5mW Thick Film Resistors ±100ppm/℃ ±1% 1kΩ 0402 Chip Resistor - Surface Mount ROHS
- R22: value 62.5mW Thick Film Resistors ±100ppm/℃ ±1% 1kΩ 0402 Chip Resistor - Surface Mount ROHS -> 62.5mW Thick Film Resistors ±100ppm/℃ ±1% 5.1kΩ 0402 Chip Resistor - Surface Mount ROHS
- R3: value 62.5mW Thick Film Resistors ±100ppm/℃ ±1% 27kΩ 0402 Chip Resistor - Surface Mount ROHS -> 62.5mW Thick Film Resistors ±100ppm/℃ ±1% 1kΩ 0402 Chip Resistor - Surface Mount ROHS
- R4, R5: value 62.5mW Thick Film Resistors ±100ppm/℃ ±1% 10kΩ 0402 Chip Resistor - Surface Mount ROHS -> 62.5mW Thick Film Resistors ±100ppm/℃ ±1% 27Ω 0402 Chip Resistor - Surface Mount ROHS
- R6: value 62.5mW Thick Film Resistors ±100ppm/℃ ±1% 510Ω 0402 Chip Resistor - Surface Mount ROHS -> 62.5mW Thick Film Resistors ±100ppm/℃ ±1% 2kΩ 0402 Chip Resistor - Surface Mount ROHS
- R7: value 62.5mW Thin Film Resistor ±0.5% ±25ppm/℃ 110Ω 0402 Chip Resistor - Surface Mount ROHS -> 62.5mW Thick Film Resistors ±100ppm/℃ ±1% 2kΩ 0402 Chip Resistor - Surface Mount ROHS
- R8: value 62.5mW Thick Film Resistors ±100ppm/℃ ±1% 82Ω 0402 Chip Resistor - Surface Mount ROHS -> 62.5mW Thick Film Resistors ±100ppm/℃ ±1% 1.07kΩ 0402 Chip Resistor - Surface Mount ROHS
- R9: value 62.5mW Thick Film Resistors ±100ppm/℃ ±1% 1MΩ 0402 Chip Resistor - Surface Mount ROHS -> 62.5mW Thick Film Resistors ±100ppm/℃ ±1% 698kΩ 0402 Chip Resistor - Surface Mount ROHS
- U10: footprint lib:LGA-16_L4.5-W3.0-P0.50-BL -> TestPoint:TestPoint_THTPad_1.0x1.0mm_Drill0.5mm
- U11: footprint lib:LGA-12_L2.0-W2.0-P0.50-BL -> lib:CONN-SMD_P2.00_S2B-PH-SM4-TB-LF-SN
- U12: footprint lib:USB-C-SMD_KH-TYPE-C-16P -> lib:WSON-10_L2.0-W2.0-P0.40-BL-EP
- U13: footprint lib:LED-SMD_4P-L2.0-W2.0-BR -> lib:VSON-14_L4.0-W3.0-P0.50-BL-EP_TI_DSJ
- U14: footprint lib:LED-SMD_4P-L2.0-W2.0-BR -> lib:SOT-223-3_L6.5-W3.4-P2.30-LS7.0-BR
- U15: footprint lib:LED-SMD_4P-L2.0-W2.0-BR -> TestPoint:TestPoint_THTPad_1.0x1.0mm_Drill0.5mm
- U16, U17, U18: footprint lib:KEY-SMD_4P-L4.2-W3.2-P2.20-LS4.6 -> TestPoint:TestPoint_THTPad_1.0x1.0mm_Drill0.5mm
- U19: footprint lib:KEY-SMD_4P-L4.2-W3.2-P2.20-LS4.6 -> lib:LGA-28_L5.2-W3.8-P0.50-BL
- U2: footprint lib:OSC-SMD_4P-L3.2-W2.5-BL -> lib:KEY-SMD_4P-L4.2-W3.2-P2.20-LS4.6
- U20: footprint lib:SOT-23-3_L2.9-W1.3-P1.90-LS2.4-BR-CW -> lib:FC-135R_L3.2-W1.5
- U3: footprint lib:SOIC-8_L5.3-W5.3-P1.27-LS8.0-BL -> lib:KEY-SMD_4P-L4.2-W3.2-P2.20-LS4.6
- U4: footprint lib:CONN-SMD_P2.00_S2B-PH-SM4-TB-LF-SN -> lib:OSC-SMD_4P-L3.2-W2.5-BL
- U5: footprint lib:WSON-10_L2.0-W2.0-P0.40-BL-EP -> lib:SOIC-8_L5.3-W5.3-P1.27-LS8.0-BL
- U6: footprint lib:VSON-14_L4.0-W3.0-P0.50-BL-EP_TI_DSJ -> TestPoint:TestPoint_THTPad_1.0x1.0mm_Drill0.5mm
- U7: footprint lib:SOT-223-3_L6.5-W3.4-P2.30-LS7.0-BR -> TestPoint:TestPoint_THTPad_1.0x1.0mm_Drill0.5mm
- U8: footprint lib:LGA-28_L5.2-W3.8-P0.50-BL -> TestPoint:TestPoint_THTPad_1.0x1.0mm_Drill0.5mm
- U9: footprint lib:FC-135R_L3.2-W1.5 -> TestPoint:TestPoint_THTPad_1.0x1.0mm_Drill0.5mm
- moved U12 168.6 mm to (185.9, 144.4), turned to 0.1 degrees
- moved C14 166.8 mm to (184.1, 143.6), turned to -89.9 degrees
- moved C22 161.7 mm to (186.1, 140.8), turned to 0.1 degrees
- moved U13 155.7 mm to (178.0, 140.6), turned to 0.1 degrees
- moved U15 155.0 mm to (175.9, 151.1)
- moved C29 144.7 mm to (181.7, 76.3), turned to -89.9 degrees
- moved R8 139.9 mm to (184.1, 145.5), turned to 90.1 degrees
- moved C15 139.2 mm to (177.5, 137.4), turned to -179.9 degrees
- moved U14 138.8 mm to (168.8, 139.7), turned to -89.9 degrees
- moved C17 137.9 mm to (177.4, 144.6), turned to -179.9 degrees
- moved C25 137.3 mm to (174.7, 76.7), turned to 0.1 degrees
- moved R13 135.5 mm to (186.1, 141.9), turned to 0.1 degrees
- moved C18 134.6 mm to (177.4, 146.6), turned to -179.9 degrees
- moved C20 134.2 mm to (173.3, 139.7), turned to 90.1 degrees
- moved C26 133.5 mm to (166.2, 80.2), turned to 0.1 degrees
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Connections:
- net gpio9 renamed micro.micro-cs
- net miso renamed micro.micro-miso
- net sck-1 renamed micro.micro-sck
- net vcc-5 renamed micro.micro.micro-vcc
- C13 pad 1: vcc-6 -> power_supply-vcc
- C14 pad 1: vcc-7 -> power_supply.battery-vcc
- C15 pad 1: vcc-7 -> power_supply.battery-vcc
- C16 pad 1: vcc-7 -> power_supply.battery-vcc
- C17 pad 1: vcc-10 -> power_supply.buckboost-vcc
- C18 pad 1: vcc-10 -> power_supply.buckboost-vcc
- C2 pad 1: out -> micro.micro.osc.osc-out
- C20 pad 1: vcc-10 -> power_supply.buckboost-vcc
- C22 pad 1: vcc -> power_supply.battery_voltage_sensor-out
- C24 pad 1: cap -> vcc
- C25 pad 1: xin32 -> cap
- C26 pad 1: xout32 -> xin32
- C27 pad 1: vcc -> xout32
- C29 pad 1: c1 -> vcc
- C30 pad 1: vcc -> gnd
- C30 pad 2: gnd -> regout
- C31 pad 1: vcc -> gnd
- C31 pad 2: gnd -> cpout
- C32 pad 1: vcc -> c1
- R1 pad 1: xout -> vcc
- R1 pad 2: out -> run
- R10 pad 1: out-1 -> power_supply.buckboost.tps_buck_boost.feedback_div-out
- R11 pad 1: pg -> power_supply.buckboost.tps_buck_boost.ic-pg
- R12 pad 1: com3 -> power_supply.battery-vcc
- R12 pad 2: gnd -> power_supply.battery_voltage_sensor-out
- R13 pad 1: ps0 -> power_supply.battery_voltage_sensor-out
- R14 pad 1: ps1 -> com3
- R15 pad 1: miso-1 -> ps0
- R16 pad 1: cc1 -> ps1
- R17 pad 1: cc2 -> interrupt
- R17 pad 2: gnd -> vcc
- R18 pad 1: vcc-15 -> micro-sda
- R18 pad 2: vcc-2 -> vcc
- R19 pad 1: vcc-16 -> micro-scl
- R19 pad 2: vcc-3 -> vcc
- R2 pad 1: usb_dp -> vcc
- R2 pad 2: dp -> micro.micro-cs-1
- R20 pad 1: vcc-17 -> imu.lis3mdltr.ic-miso
- R20 pad 2: vcc-4 -> gnd
- R21 pad 1: vcc-18 -> vcc
- R21 pad 2: tx -> radio._micro.ic-en
- R22 pad 1: vcc -> radio.usbconn.conn-cc1
- R22 pad 2: vcc-11 -> gnd
- R3 pad 1: dm -> xout
- R3 pad 2: usb_dm -> micro.micro.osc.osc-out
- R4 pad 1: vcc -> usb_dp
- R4 pad 2: run -> micro-dp
- R5 pad 1: vcc -> micro-dm
- R5 pad 2: cs -> usb_dm
- R6 pad 1: iset -> micro-sda
- R6 pad 2: gnd -> vcc
- R7 pad 1: cathode -> micro-scl
- R7 pad 2: gnd-5 -> vcc
- R8 pad 1: cathode-1 -> iset
- R8 pad 2: gnd-6 -> gnd
- R9 pad 1: vcc-10 -> power_supply.buckboost-vcc
- R9 pad 2: out-1 -> power_supply.buckboost.tps_buck_boost.feedback_div-out
- U1 pad 15: gpio12 -> micro-vcc-1
- U1 pad 16: gpio13 -> micro-vcc-2
- U1 pad 2: vcc-1 -> gpio0
- U1 pad 28: gpio17 -> micro-vcc-5
- U1 pad 3: vcc-2 -> gpio1
- U1 pad 31: sda -> micro-sda
- U1 pad 32: scl -> micro-scl
- U1 pad 36: gpio24 -> micro-vcc
- U1 pad 38: gpio26_a0 -> micro-vcc-4
- U1 pad 4: vcc-3 -> gpio2
- U1 pad 5: vcc-4 -> gpio3
- U1 pad 51: io3 -> micro.micro-io3
- U1 pad 52: sck -> micro.micro-sck-1
- U1 pad 53: io0 -> micro.micro-io0
- U1 pad 54: io2 -> micro.micro-io2
- U1 pad 55: io1 -> micro.micro-io1
- U1 pad 56: cs -> micro.micro-cs-1
- U1 pad 9: gpio7 -> micro-vcc-3
- U10 pad 1: int2 -> micro-vcc
- U11 pad 1: scl -> gnd
- U11 pad 2: gnd -> power_supply.battery-vcc
- U11 pad 3: gnd -> (no net)
- U11 pad 4: c1 -> (no net)
- U12 pad 1: gnd -> power_supply-vcc
- U12 pad 2: gnd -> iset
- U12 pad 4: gnd -> preterm
- U13 pad 1: vcc -> vina
- U13 pad 2: vcc-12 -> gnd
- U13 pad 3: gnd -> power_supply.buckboost.tps_buck_boost.feedback_div-out
- U13 pad 4: rx -> power_supply.buckboost-vcc
- U14 pad 1: vcc -> gnd
- U14 pad 2: vcc-13 -> vcc
- U14 pad 3: gnd -> power_supply.buckboost-vcc
- U14 pad 4: vcc-12 -> vcc
- U15 pad 1: vcc -> power_supply-vcc
- U16 pad 1: vcc-2 -> vcc
- U17 pad 1: vcc-3 -> power_supply.battery-vcc
- U18 pad 1: vcc-4 -> micro-vcc-5
- U19 pad 1: tx -> pin1
- U19 pad 2: tx -> gnd
- U19 pad 3: gnd -> vcc
- U19 pad 4: gnd -> vcc
- U2 pad 1: xin -> run
- U2 pad 2: gnd -> run
- U2 pad 3: out -> gnd
- U20 pad 1: vcc -> xin32
- U20 pad 2: gnd -> xout32
- U3 pad 1: cs -> micro.micro-cs-1
- U3 pad 2: io1 -> micro.micro-cs-1
- U3 pad 3: io2 -> gnd
- U4 pad 1: gnd -> xin
- U4 pad 2: vcc-7 -> gnd
- U4 pad 3: (no net) -> micro.micro.osc.osc-out
- U4 pad 4: (no net) -> gnd
- U5 pad 1: vcc-6 -> micro.micro-cs-1
- U5 pad 2: iset -> micro.micro-io1
- U5 pad 3: gnd -> micro.micro-io2
- U5 pad 4: preterm -> gnd
- U5 pad 5: gnd-5 -> micro.micro-io0
- U5 pad 6: nc -> micro.micro-sck-1
- U5 pad 7: vcc-6 -> micro.micro-io3
- U5 pad 8: gnd-6 -> vcc
- U6 pad 1: vina -> micro-scl
- U7 pad 1: gnd -> micro-sda
- U8 pad 1: pin1 -> tx
- U9 pad 1: xin32 -> rx
Routing:
- net gnd: track 0.00 -> 245.1 mm, vias 0 -> 92
- net vcc: track 0.00 -> 163.2 mm, vias 0 -> 28
- net micro-sda: track 0.00 -> 158.5 mm, vias 0 -> 7
- net micro-scl: track 0.00 -> 154.6 mm, vias 0 -> 7
- net micro-dp: track 0.00 -> 80.4 mm, vias 0 -> 2
- net radio._micro.ic-scl: track 0.00 -> 76.7 mm, vias 0 -> 4
- net micro-dm: track 0.00 -> 74.8 mm, vias 0 -> 2
- net micro-vcc-4: track 0.00 -> 72.0 mm, vias 0 -> 2
- net radio._micro.ic-sda: track 0.00 -> 69.8 mm, vias 0 -> 2
- net micro-vcc-5: track 0.00 -> 63.7 mm, vias 0 -> 2
- net micro-vcc-1: track 0.00 -> 61.3 mm, vias 0 -> 1
- net micro-vcc-3: track 0.00 -> 55.0 mm, vias 0 -> 3
- net micro-vcc-2: track 0.00 -> 53.9 mm, vias 0 -> 1
- net ios.led1.ic-vcc: track 0.00 -> 51.6 mm
- net radio._micro.ic-dp: track 0.00 -> 37.4 mm, vias 0 -> 2
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- added copper zone on F.Cu, net gnd
- added copper zone on In1.Cu, net gnd
- added copper zone on B.Cu, net vcc
- added copper zone on In2.Cu, net vcc
Other:
- board size 100 x 100 mm -> 80 x 131.9 mm
- copper layers 2 -> 4
- board text added: "3v3"
- board text added: "I2C"
- board text added: "LCD"
- board text added: "MAG"
- board text added: "Menu"
- board text added: "Power"
- board text added: "RX"
- board text added: "SCL"
- board text added: "SDA"
- board text added: "SWOOP"
- board text added: "TX"
- board text added: "ba64ff3"
- board text removed: "{{GITHASH}}"

Commit message: cleaner commit
Parts:
- removed J2: , lib:CONN-SMD_4P-P1.00_SM04B-SRSS-TB-LF-SN
- removed the R22 at (176.3, 87.1)
- removed the R23 at (175.9, 84.1)
- removed the R24 at (162.4, 70.5)
- removed the R25 at (161.3, 70.5)
- removed the U29 at (180.7, 85.4)
- C1, C2: value 50V 20pF C0G ±5% 0402 Multilayer Ceramic Capacitors MLCC - SMD/SMT ROHS -> 50V 18pF C0G ±5% 0402 Multilayer Ceramic Capacitors MLCC - SMD/SMT ROHS
- C26, C27: value 50V 22pF C0G ±5% 0402 Multilayer Ceramic Capacitors MLCC - SMD/SMT ROHS -> 50V 18pF C0G ±5% 0402 Multilayer Ceramic Capacitors MLCC - SMD/SMT ROHS
- C38, C39: value 50V 11pF C0G ±5% 0402 Multilayer Ceramic Capacitors MLCC - SMD/SMT ROHS -> 50V 12pF C0G ±5% 0402 Multilayer Ceramic Capacitors MLCC - SMD/SMT ROHS
- C40: value 10V 470nF X5R ±10% 0402 Multilayer Ceramic Capacitors MLCC - SMD/SMT ROHS -> 50V 470nF X5R ±10% 0402 Multilayer Ceramic Capacitors MLCC - SMD/SMT ROHS
- C45: value 50V 1pF C0G 0402 Multilayer Ceramic Capacitors MLCC - SMD/SMT ROHS -> 50V 0.8pF 0402 Multilayer Ceramic Capacitors MLCC - SMD/SMT ROHS
- C46, C47: value 50V 1pF C0G 0402 Multilayer Ceramic Capacitors MLCC - SMD/SMT ROHS -> 50V 1.2pF C0G 0402 Multilayer Ceramic Capacitors MLCC - SMD/SMT ROHS
- C48: value 50V 1pF C0G 0402 Multilayer Ceramic Capacitors MLCC - SMD/SMT ROHS -> 50V 0.5pF C0G 0402 Multilayer Ceramic Capacitors MLCC - SMD/SMT ROHS
- R1, R17, R18, R19, R2, R21: value 62.5mW Thick Film Resistors ±100ppm/℃ ±1% 10kΩ 0402 Chip Resistor - Surface Mount ROHS -> 62.5mW Thick Film Resistors 50V ±100ppm/℃ ±1% 10kΩ 0402 Chip Resistor - Surface Mount ROHS
- R10: value 62.5mW Thick Film Resistors ±100ppm/℃ ±1% 105kΩ 0402 Chip Resistor - Surface Mount ROHS -> 62.5mW Thick Film Resistors 50V ±1% ±200ppm/℃ 105kΩ 0402 Chip Resistor - Surface Mount ROHS
- R11: value 62.5mW Thick Film Resistors ±100ppm/℃ ±1% 1MΩ 0402 Chip Resistor - Surface Mount ROHS -> 62.5mW Thick Film Resistors 50V ±100ppm/℃ ±1% 1MΩ 0402 Chip Resistor - Surface Mount ROHS
- R12: value 62.5mW Thick Film Resistors ±100ppm/℃ ±1% 16.2kΩ 0402 Chip Resistor - Surface Mount ROHS -> 62.5mW Thick Film Resistors 50V ±100ppm/℃ ±1% 16.2kΩ 0402 Chip Resistor - Surface Mount ROHS
- R13: value 62.5mW Thick Film Resistors ±100ppm/℃ ±1% 17.8kΩ 0402 Chip Resistor - Surface Mount ROHS -> 62.5mW Thick Film Resistors 50V ±100ppm/℃ ±1% 17.8kΩ 0402 Chip Resistor - Surface Mount ROHS
- R14, R15, R16: value 62.5mW Thick Film Resistors ±1% ±400ppm/℃ 5.1Ω 0402 Chip Resistor - Surface Mount ROHS -> 62.5mW Thick Film Resistors 50V ±100ppm/℃ ±1% 10kΩ 0402 Chip Resistor - Surface Mount ROHS
- R20, R3: value 62.5mW Thick Film Resistors ±100ppm/℃ ±1% 1kΩ 0402 Chip Resistor - Surface Mount ROHS -> 62.5mW Thick Film Resistors 50V ±100ppm/℃ ±1% 1kΩ 0402 Chip Resistor - Surface Mount ROHS
- R22: renamed from R26; value 62.5mW Thick Film Resistors ±100ppm/℃ ±1% 10kΩ 0402 Chip Resistor - Surface Mount ROHS -> 62.5mW Thick Film Resistors 50V ±100ppm/℃ ±1% 10kΩ 0402 Chip Resistor - Surface Mount ROHS
- R23: renamed from R27; value 62.5mW Thick Film Resistors ±100ppm/℃ ±1% 5.1kΩ 0402 Chip Resistor - Surface Mount ROHS -> 62.5mW Thick Film Resistors 50V ±100ppm/℃ ±1% 4.7kΩ 0402 Chip Resistor - Surface Mount ROHS
- R24: renamed from R28; value 62.5mW Thick Film Resistors ±100ppm/℃ ±1% 5.1kΩ 0402 Chip Resistor - Surface Mount ROHS -> 62.5mW Thick Film Resistors 50V ±100ppm/℃ ±1% 4.7kΩ 0402 Chip Resistor - Surface Mount ROHS
- R25: renamed from R29; value 62.5mW Thick Film Resistors ±100ppm/℃ ±1% 10kΩ 0402 Chip Resistor - Surface Mount ROHS -> 62.5mW Thick Film Resistors 50V ±100ppm/℃ ±1% 10kΩ 0402 Chip Resistor - Surface Mount ROHS
- R26: renamed from R30; value 62.5mW Thick Film Resistors ±100ppm/℃ ±1% 10kΩ 0402 Chip Resistor - Surface Mount ROHS -> 62.5mW Thick Film Resistors 50V ±100ppm/℃ ±1% 10kΩ 0402 Chip Resistor - Surface Mount ROHS
- R4, R5: value 62.5mW Thick Film Resistors ±100ppm/℃ ±1% 27Ω 0402 Chip Resistor - Surface Mount ROHS -> 62.5mW Thick Film Resistors 50V ±100ppm/℃ ±1% 27Ω 0402 Chip Resistor - Surface Mount ROHS
- R6, R7: value 62.5mW Thick Film Resistors ±100ppm/℃ ±1% 2kΩ 0402 Chip Resistor - Surface Mount ROHS -> 62.5mW Thick Film Resistors 50V ±100ppm/℃ ±1% 2kΩ 0402 Chip Resistor - Surface Mount ROHS
- R8: value 62.5mW Thick Film Resistors ±100ppm/℃ ±1% 1.07kΩ 0402 Chip Resistor - Surface Mount ROHS -> 100mW Thick Film Resistors ±100ppm/℃ ±1% 1.07kΩ 0402 Chip Resistor - Surface Mount ROHS
- R9: value 62.5mW Thick Film Resistors ±100ppm/℃ ±1% 698kΩ 0402 Chip Resistor - Surface Mount ROHS -> 62.5mW Thick Film Resistors 50V ±100ppm/℃ ±1% 698kΩ 0402 Chip Resistor - Surface Mount ROHS
- renumbered R31 to R27, U30 to U29, U31 to U30, U32 to U31, U33 to U32, U34 to U33, U35 to U34, U36 to U35, U37 to U36, U38 to U37, U39 to U38, U40 to U39, U41 to U40
Connections:
- net ios.usbc_connector.conn-cc1 renamed cc1
- net ios.usbc_connector.conn-cc2 renamed cc2
- net ios.usbc_connector.conn-sub1 renamed sub1
- net ios.usbc_connector.conn-sub2 renamed sub2
- net micro-dm renamed dm
- net micro-dp renamed dp
- net micro-scl renamed scl
- net micro-sda renamed sda
- net radio._micro.ic-io renamed io
- net radio._micro.ic-scl renamed io6
- net radio._micro.ic-sda renamed io7
- net radio._radio.ic-io renamed radio._radio.ic-vcc-2
- U21 pad 14: vcc -> csb1
- U21 pad 15: sdo1 -> sdo2
- U24 pad 13: radio._micro.ic-dm -> io19
- U24 pad 14: radio._micro.ic-dp -> io20
Routing:
- net radio._micro.ic-dp: track 37.4 -> 0.00 mm, vias 2 -> 0
- net io20: track 0.00 -> 37.4 mm, vias 0 -> 2
- net radio._micro.ic-dm: track 34.8 -> 0.00 mm, vias 2 -> 0
- net io19: track 0.00 -> 34.8 mm, vias 0 -> 2
- net (no net): track 0.00 -> 12.6 mm
- net radio.usbconn-vcc: track 9.31 -> 0.00 mm
- net radio.usbconn.conn-cc2: track 1.65 -> 0.00 mm
- net radio.usbconn.conn-cc1: track 1.60 -> 0.00 mm
