File: elec/layout/debug/debug.kicad_pcb (KiCad board)
At the start: 4 copper layers, 100 x 100 mm, 150 parts

Commit message: merging in layouts
Parts:
- removed the U4 at (249.6, 78.8)
- removed the U5 at (241.5, 81.8)
- added U2: , lib:OSC-SMD_4P-L3.2-W2.5-BL, F.Cu at (152.0, 119.4)
- added U3: , lib:SOIC-8_L5.3-W5.3-P1.27-LS8.0-BL, F.Cu at (134.8, 118.0)
- R3: value 62.5mW Thick Film Resistors ±100ppm/℃ ±1% 10kΩ 0402 Chip Resistor - Surface Mount ROHS -> 62.5mW Thick Film Resistors ±100ppm/℃ ±1% 1kΩ 0402 Chip Resistor - Surface Mount ROHS
- R4: value 62.5mW Thick Film Resistors ±100ppm/℃ ±1% 10kΩ 0402 Chip Resistor - Surface Mount ROHS -> 62.5mW Thick Film Resistors ±100ppm/℃ ±1% 27kΩ 0402 Chip Resistor - Surface Mount ROHS
- R5: value 62.5mW Thick Film Resistors ±100ppm/℃ ±1% 1kΩ 0402 Chip Resistor - Surface Mount ROHS -> 62.5mW Thick Film Resistors ±100ppm/℃ ±1% 27kΩ 0402 Chip Resistor - Surface Mount ROHS
- R6, R7: value 62.5mW Thick Film Resistors ±100ppm/℃ ±1% 27kΩ 0402 Chip Resistor - Surface Mount ROHS -> 62.5mW Thick Film Resistors ±100ppm/℃ ±1% 10kΩ 0402 Chip Resistor - Surface Mount ROHS
- moved C5 127.5 mm to (139.6, 123.3), turned to -90 degrees
- moved C8 126.3 mm to (131.7, 114.3), turned to -90 degrees
- moved C7 124.8 mm to (144.5, 112.5), turned to 90 degrees
- moved C9 123.6 mm to (138.5, 118.0), turned to 180 degrees
- moved R4 123.4 mm to (137.8, 114.3), turned to 90 degrees
- moved C10 122.8 mm to (139.9, 112.6), turned to 90 degrees
- moved C4 122.6 mm to (141.0, 112.6), turned to 90 degrees
- moved C12 118.3 mm to (150.8, 114.6)
- moved R6 117.1 mm to (144.8, 123.3), turned to -90 degrees
- moved C11 115.9 mm to (150.8, 115.6)
- moved C3 115.2 mm to (150.8, 116.7)
- moved C2 114.7 mm to (152.7, 116.7)
- moved R7 114.2 mm to (138.9, 121.3), turned to 90 degrees
- moved R5 113.3 mm to (138.9, 114.3), turned to -90 degrees
- moved R3 112.1 mm to (149.7, 118.2), turned to 90 degrees
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- renumbered U2 to U4, U3 to U5
Connections:
- net cs-3 renamed cs-2
- R3 pad 1: vcc -> xout
- R3 pad 2: run -> out
- R4 pad 1: vcc -> usb_dp
- R4 pad 2: cs-1 -> dp
- R5 pad 1: xout -> dm
- R5 pad 2: out -> usb_dm
- R6 pad 1: dp -> vcc
- R6 pad 2: dp -> run
- R7 pad 1: dm -> vcc
- R7 pad 2: dm -> cs
- U1 pad 12: cs -> gpio9
- U1 pad 13: sck -> sck-1
- U1 pad 43: adc_avdd -> vcc
- U1 pad 46: dm -> usb_dm
- U1 pad 47: dp -> usb_dp
- U1 pad 48: usb_vdd -> vcc
- U1 pad 52: sck-1 -> sck
- U1 pad 56: cs-1 -> cs
- U5 pad 1: cs-1 -> cs
- U5 pad 2: cs-1 -> cs
Routing:
- net vcc: track 94.4 -> 136.9 mm, vias 32 -> 35
- net vcc-8: track 0.00 -> 23.4 mm, vias 0 -> 2
- net cs: track 0.00 -> 18.1 mm
- net sck: track 0.00 -> 14.4 mm
- net io0: track 0.00 -> 12.8 mm, vias 0 -> 2
- net io3: track 0.00 -> 9.73 mm
- net io1: track 0.00 -> 9.57 mm
- net xin: track 0.00 -> 8.08 mm
- net io2: track 0.00 -> 6.20 mm
- net gnd: track 205.6 -> 211.0 mm, vias 62 -> 65
- net cs-1: track 4.35 -> 0.00 mm
- net run: track 15.5 -> 19.7 mm
- net vcc-1: track 136.8 -> 141.0 mm
- net usb_dp: track 0.00 -> 4.15 mm
- net out: track 0.00 -> 3.72 mm
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